File: boards/445project.kicad_sch (KiCad schematic)
At the start: 29 parts, among them J1 ULTRASONIC_2, J10 RGB_FLASH, J2 ULTRASONIC_1, J3 M1, J4 M2, J5 Buzzer, J6 PI1, J7 PI2, J8 PI3, J9 Camera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

Commit message: pcb version 1
Parts:
- removed P1: USB_C_Plug_USB2.0, Connector_USB:USB_C_Plug_Molex_105444, symbol Connector:USB_C_Plug_USB2.0
- added J11: USB_C_Receptacle_USB2.0_14P, Connector_USB:USB_C_Receptacle_GCT_USB4105-xx-A_16P_TopMnt_Horizontal, symbol Connector:USB_C_Receptacle_USB2.0_14P
Connections:
- net +5V: now also J11.A4 (VBUS), J11.A9 (VBUS), J11.B4 (VBUS), J11.B9 (VBUS)
- net GND: now also J11.A1 (GND), J11.A12 (GND), J11.B1 (GND), J11.B12 (GND), J11.S1 (SHIELD)
- net USB_N: now also J11.A7 (D-), J11.B7 (D-)
- net USB_P: now also J11.A6 (D+), J11.B6 (D+)
- net at R1.1: now also J11.A5 (CC1)
- net at R2.1: now also J11.B5 (CC2)
Changed lines of the file:
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@@
   (junction (at 113.03 102.87) (diameter 0) (color 0 0 0 0)
   )
+  (junction (at 46.99 43.18) (diameter 0) (color 0 0 0 0)
+  )
   (junction (at 77.47 185.42) (diameter 0) (color 0 0 0 0)
   )
@@
   (junction (at 77.47 161.29) (diameter 0) (color 0 0 0 0)
   )
+  (junction (at 46.99 38.1) (diameter 0) (color 0 0 0 0)
+  )
   (junction (at 81.28 25.4) (diameter 0) (color 0 0 0 0)
   )
@@
     (stroke (width 0) (type default))
   )
+  (wire (pts (xy 46.99 43.18) (xy 46.99 45.72))
+    (stroke (width 0) (type default))
+  )
   (wire (pts (xy 53.34 30.48) (xy 60.96 30.48))
     (stroke (width 0) (type default))
@@
   )
   (wire (pts (xy 172.72 82.55) (xy 172.72 81.28))
+    (stroke (width 0) (type default))
+  )
+  (wire (pts (xy 46.99 38.1) (xy 46.99 40.64))
     (stroke (width 0) (type default))
   )
@@
     )
   )
+  (symbol (lib_id "Connector:USB_C_Receptacle_USB2.0_14P") (at 31.75 40.64 0) (unit 1)
+    (in_bom yes) (on_board yes) (dnp no) (fields_autoplaced)
+    (property "Reference" "J11" (at 31.75 17.78 0)
+      (effects (font (size 1.27 1.27)))
+    )
+    (property "Value" "USB_C_Receptacle_USB2.0_14P" (at 31.75 20.32 0)
+      (effects (font (size 1.27 1.27)))
+    )
+    (property "Footprint" "Connector_USB:USB_C_Receptacle_GCT_USB4105-xx-A_16P_TopMnt_Horizontal" (at 35.56 40.64 0)
+      (effects (font (size 1.27 1.27)) hide)
+    )
+    (property "Datasheet" "https://www.usb.org/sites/default/files/documents/usb_type-c.zip" (at 35.56 40.64 0)
+      (effects (font (size 1.27 1.27)) hide)
+    )
+    (pin "A7")
+    (pin "A9")
+    (pin "S1")
+    (pin "B4")
+    (pin "A5")
+    (pin "A6")
+    (pin "A12")
+    (pin "B5")
+    (pin "B9")
+    (pin "A1")
+    (pin "B1")
+    (pin "B12")
+    (pin "B6")
+    (pin "A4")
+    (pin "B7")
+    (instances
+      (project "445project"
+        (path "/e63e39d7-6ac0-4ffd-8aa3-1841a4541b55"
+          (reference "J11") (unit 1)
+        )
+      )
+    )
+  )
   (symbol (lib_id "Connector_Generic:Conn_01x06") (at 254 90.17 0) (unit 1)
     (in_bom yes) (on_board yes) (dnp no) (fields_autoplaced)
@@
         )
       )
-    )
-  )
-  (symbol (lib_id "Connector:USB_C_Plug_USB2.0") (at 31.75 40.64 0) (unit 1)
-    (in_bom yes) (on_board yes) (dnp no) (fields_autoplaced)
-    (property "Reference" "P1" (at 31.75 17.78 0)
-      (effects (font (size 1.27 1.27)))
-    )
-    (property "Value" "USB_C_Plug_USB2.0" (at 31.75 20.32 0)
-      (effects (font (size 1.27 1.27)))
-    )
-    (property "Footprint" "Connector_USB:USB_C_Plug_Molex_105444" (at 35.56 40.64 0)
-      (effects (font (size 1.27 1.27)) hide)
-    )
-    (property "Datasheet" "https://www.usb.org/sites/default/files/documents/usb_type-c.zip" (at 35.56 40.64 0)
-      (effects (font (size 1.27 1.27)) hide)
-    )
-    (pin "A4")
-    (pin "B1")
-    (pin "A7")
-    (pin "B4")
-    (pin "A6")
-    (pin "B12")
-    (pin "A1")
-    (pin "S1")
-    (pin "B9")
-    (pin "A12")
-    (pin "A5")
-    (pin "A9")
-    (pin "B5")
-    (instances
-      (project "445project"
-        (path "/e63e39d7-6ac0-4ffd-8aa3-1841a4541b55"
-          (reference "P1") (unit 1)
-        )
-      )
